File: sm/sm.kicad_sch (KiCad schematic)
At the start: 165 parts, among them M1 TPS61040, M2 LM5164, M3 STM32F405RG, M4 TPS73633, M5 UCC27211A, M6 UCC27211A, M7 UCC27211A, M8 SN65HVD256, P1 USART, P2 SWD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

Commit message: Trace tracks
Select components
Parts:
- removed R43, R44: 0.0005 1%, Resistor_SMD:R_Shunt_Vishay_WSK2512_6332Metric_T1.19mm, symbol fake:R-4
- added R43, R44: 0.0005 1%, Resistor_SMD:R_Shunt_Vishay_WSK2512_6332Metric_T1.19mm, symbol Device:R_Shunt
- C1, C3: LCSC (none) -> C153036; MFR PT (none) -> FS32X225K101EGG
- C10: LCSC (none) -> C92834; MFR PT (none) -> TMK325BJ106KN-T
- C11: LCSC (none) -> C36576; MFR PT (none) -> 0805B222K500NT
- C12, C9: LCSC (none) -> C107034; MFR PT (none) -> CC0603JRNPO9BN120
- C13, C16, C17, C24, C26, C31, C32, C33, C34, C35, C39, C4, C41, C43, C47, C49, C51, C56, C57, C58, C6, C65, C66: LCSC (none) -> C519981; MFR PT (none) -> CC0805KRX7R8BB104
- C14, C15: LCSC (none) -> C107041; MFR PT (none) -> CC0603JRNPO9BN181
- C18, C27, C28, C29, C36, C37, C64, C7, C8: LCSC (none) -> C285099; MFR PT (none) -> 0603B103K250NT
- C19, C40, C42, C44, C59: LCSC (none) -> C713511; MFR PT (none) -> TCC0805X5R105M250FT
- C2, C22, C23, C25, C30: LCSC (none) -> C92762; MFR PT (none) -> EMK212B7475KG-T
- C20, C21: LCSC (none) -> C5189825; MFR PT (none) -> CS3225X7R476K100NRL
- C46, C48, C50: LCSC (none) -> C1779; MFR PT (none) -> CL21A475KAQNNNE
- C5: LCSC (none) -> C28233; MFR PT (none) -> CL21B104KCFNNNE
- C52, C53, C54, C55: LCSC (none) -> C6120033; MFR PT (none) -> CGA1210X7R475K101RT
- C60, C61, C62, C63: LCSC (none) -> C163508; MFR PT (none) -> CL10C102JB8NNNC
- D1: LCSC (none) -> C19171392; MFR PT (none) -> YLED0603YG
- D3: LCSC (none) -> C109001; MFR PT (none) -> CD4148WSP
- L1: LCSC C7529415 -> C7529415
- L2: LCSC (none) -> C7461363; MFR PT (none) -> CXP0630-220M-AG(22uh)
- M1: LCSC (none) -> C7722; MFR PT (none) -> TPS61040DBVR
- M2: LCSC C477928 -> C477928
- M3: LCSC C15742 -> C15742
- M4: LCSC (none) -> C28038; MFR PT (none) -> TPS73633DBVR
- M5, M6, M7: LCSC (none) -> C485921; MFR PT (none) -> UCC27211AQDDARQ1
- M8: LCSC (none) -> C132551; MFR PT (none) -> SN65HVD256DR
- P1, P5, P6: LCSC (none) -> C265289; MFR PT (none) -> B4B-PH-K(LF)(SN)
- P2, P7, P8, P9: LCSC (none) -> C5251182; MFR PT (none) -> B2B-PH-K-S-GW
- P3: LCSC (none) -> C157993; MFR PT (none) -> B5B-PH-K-S(LF)(SN)
- P4: LCSC (none) -> C495261; MFR PT (none) -> B6B-PH-K-S-GW
- Q1, Q2, Q3, Q4, Q5, Q6: LCSC (none) -> C3288766; MFR PT (none) -> IPT010N08NM5ATMA1
- Q7: LCSC C2835446 -> C2835446
- R1: LCSC (none) -> C22809; MFR PT (none) -> 0603WAF1502T5E
- R10: LCSC (none) -> C22793; MFR PT (none) -> 0603WAF1372T5E
- R11, R12, R13, R2, R33, R34, R35, R36, R59: LCSC (none) -> C25804; MFR PT (none) -> 0603WAF1002T5E
- R14, R15, R16, R17, R18, R19, R20, R21, R26, R27, R4: LCSC (none) -> C23138; MFR PT (none) -> 0603WAF3300T5E
- R22, R3: LCSC (none) -> C22936; MFR PT (none) -> 0603WAF100KT5E
- R23, R24, R25, R28, R29, R30, R31, R32, R46, R5, R6: LCSC (none) -> C21190; MFR PT (none) -> 0603WAF1001T5E
- R37, R38, R39, R40, R41, R42: LCSC (none) -> C22977; MFR PT (none) -> 0603WAF200KT5E
- R45: LCSC (none) -> C25819; MFR PT (none) -> 0603WAF4702T5E
- R47: LCSC (none) -> C4502; MFR PT (none) -> 1206W4F4700T5E
- R48, R49, R50, R51, R56, R57, R58: LCSC (none) -> C23178; MFR PT (none) -> 0603WAF4703T5E
- R52, R53, R54, R55: LCSC (none) -> C31850; MFR PT (none) -> 0603WAF2202T5E
- R60: LCSC (none) -> C95968; MFR PT (none) -> SDNT2012X103F3950FTF
- R7: LCSC (none) -> C25967; MFR PT (none) -> 0603WAF3162T5E
- R8, R9: LCSC (none) -> C25803; MFR PT (none) -> 0603WAF1003T5E
- U1, U2: LCSC (none) -> C495342; MFR PT (none) -> AD8418WBRZ-RL
- U3, U4: LCSC (none) -> C154930; MFR PT (none) -> AD8539ARZ-REEL7
- Z1: LCSC (none) -> C9002; MFR PT (none) -> X322512MSB4SI
Connections:
- net TERMINAL_A: now also R43.4
- net TERMINAL_B: now also R44.4
- net at C48.1, C49.1, M6.4 (HS)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: now also R44.1
- net at C46.1, C47.1, M5.4 (HS)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: now also R43.1
- net at U1.8 (+): now also R43.2
- net at U1.1 (_): now also R43.3
- net at U2.1 (_): now also R44.3
- net at U2.8 (+): now also R44.2
Other:
- moved on the sheet: Q1

Commit message: fix errors
Parts:
- U1, U2, U3, U4: footprint Package_SO:SOIC-8-N7_3.9x4.9mm_P1.27mm -> Package_SO:SOIC-8_3.9x4.9mm_P1.27mm
Changed lines of the file:
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@@
 			)
 		)
-		(property "Footprint" "Package_SO:SOIC-8-N7_3.9x4.9mm_P1.27mm"
+		(property "Footprint" "Package_SO:SOIC-8_3.9x4.9mm_P1.27mm"
 			(at 746.76 83.82 0)
 			(effects
@@
 					(size 1.524 1.524)
 				)
+				(hide yes)
 			)
 		)
@@
 					(size 1.524 1.524)
 				)
+				(hide yes)
 			)
 		)
@@
 					(size 1.524 1.524)
 				)
+				(hide yes)
 			)
 		)
@@
 					(size 1.524 1.524)
 				)
+				(hide yes)
 			)
 		)
@@
 					(size 1.524 1.524)
 				)
+				(hide yes)
 			)
 		)
@@
 			)
 		)
-		(property "Footprint" "Package_SO:SOIC-8-N7_3.9x4.9mm_P1.27mm"
+		(property "Footprint" "Package_SO:SOIC-8_3.9x4.9mm_P1.27mm"
 			(at 574.04 59.69 0)
 			(effects
@@
 					(size 1.524 1.524)
 				)
+				(hide yes)
 			)
 		)
@@
 					(size 1.524 1.524)
 				)
+				(hide yes)
 			)
 		)
@@
 					(size 1.524 1.524)
 				)
+				(hide yes)
 			)
 		)
@@
 			)
 		)
-		(property "Footprint" "Package_SO:SOIC-8-N7_3.9x4.9mm_P1.27mm"
+		(property "Footprint" "Package_SO:SOIC-8_3.9x4.9mm_P1.27mm"
 			(at 574.04 110.49 0)
 			(effects
@@
 					(size 1.524 1.524)
 				)
+				(hide yes)
 			)
 		)
@@
 					(size 1.524 1.524)
 				)
+				(hide yes)
 			)
 		)
@@
 			)
 		)
-		(property "Footprint" "Package_SO:SOIC-8-N7_3.9x4.9mm_P1.27mm"
+		(property "Footprint" "Package_SO:SOIC-8_3.9x4.9mm_P1.27mm"
 			(at 746.76 49.53 0)
 			(effects
@@
 					(size 1.524 1.524)
 				)
+				(hide yes)
 			)
 		)
@@
 					(size 1.524 1.524)
 				)
+				(hide yes)
 			)
 		)
@@
 					(size 1.524 1.524)
 				)
+				(hide yes)
 			)
 		)
@@
 			)
 		)
-		(property "Footprint" "Package_SO:SOIC-8-N7_3.9x4.9mm_P1.27mm"
+		(property "Footprint" "Package_SO:SOIC-8_3.9x4.9mm_P1.27mm"
 			(at 746.76 152.4 0)
 			(effects
@@
 					(size 1.524 1.524)
 				)
+				(hide yes)
 			)
 		)
@@
 			)
 		)
-		(property "Footprint" "Package_SO:SOIC-8-N7_3.9x4.9mm_P1.27mm"
+		(property "Footprint" "Package_SO:SOIC-8_3.9x4.9mm_P1.27mm"
 			(at 746.76 118.11 0)
 			(effects
@@
 					(size 1.524 1.524)
 				)
+				(hide yes)
 			)
 		)
@@
 					(size 1.524 1.524)
 				)
+				(hide yes)
 			)
 		)
@@
 					(size 1.524 1.524)
 				)
+				(hide yes)
 			)
 		)
@@
 					(size 1.524 1.524)
 				)
+				(hide yes)
 			)
 		)
