File: sm/sm.kicad_pcb (KiCad board)
At the start: 2 copper layers, 84.4 x 122.2 mm, 165 parts, among them M1 TPS61040, M2 LM5164, M3 STM32F405RG, M4 TPS73633, M5 UCC27211A, M6 UCC27211A, M7 UCC27211A, M8 SN65HVD256, P1 USART, P2 SWD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

Commit message: fix errors
Parts:
- U1, U2, U3, U4: footprint Package_SO:SOIC-8-N7_3.9x4.9mm_P1.27mm -> Package_SO:SOIC-8_3.9x4.9mm_P1.27mm
Connections:
- M5 pad 9: GND -> (no net)
- M6 pad 9: GND -> (no net)
- M7 pad 9: GND -> (no net)
Routing:
- net GND: track 444.6 -> 432.0 mm
- net +3.3V: track 307.4 -> 311.3 mm
- net VOLTAGE_A: track 23.3 -> 25.0 mm
- net VOLTAGE_U: track 10.5 -> 11.8 mm
- net VOLTAGE_C: track 25.9 -> 27.2 mm

Commit message: Fix pcbs
Routing:
- net CURRENT_B: track 75.4 -> 76.2 mm
Changed lines of the file:
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@@
 		(tags "SOIC SO")
 		(property "Reference" "U4"
-			(at 0 -3.4 90)
+			(at -1.05 -4.645 90)
 			(layer "F.SilkS")
 			(effects
@@
 	)
 	(segment
-		(start 142.748 63.9572)
-		(end 142.748 72.036604)
-		(width 0.25)
+		(start 135.636 34.798)
+		(end 131.0071 30.1691)
+		(width 0.5)
 		(layer "B.Cu")
 		(net 1)
 	)
 	(segment
-		(start 135.636 34.798)
-		(end 131.0071 30.1691)
-		(width 0.5)
+		(start 142.748 71.248)
+		(end 153.3 81.8)
+		(width 0.25)
 		(layer "B.Cu")
 		(net 1)
@@
 	)
 	(segment
-		(start 142.748 72.036604)
-		(end 152.511396 81.8)
-		(width 0.25)
+		(start 131.0071 30.1691)
+		(end 116.287576 30.1691)
+		(width 0.5)
 		(layer "B.Cu")
 		(net 1)
 	)
 	(segment
-		(start 152.511396 81.8)
-		(end 167.6872 81.8)
+		(start 142.748 63.9572)
+		(end 142.748 71.248)
 		(width 0.25)
 		(layer "B.Cu")
@@
 	)
 	(segment
-		(start 131.0071 30.1691)
-		(end 116.287576 30.1691)
-		(width 0.5)
+		(start 153.3 81.8)
+		(end 167.6872 81.8)
+		(width 0.25)
 		(layer "B.Cu")
 		(net 1)
@@
 	)
 	(segment
-		(start 145.75 71.15)
-		(end 145.75 73.8138)
-		(width 0.25)
-		(layer "F.Cu")
-		(net 32)
-	)
-	(segment
 		(start 112.3 117.6)
 		(end 114.35 117.6)
@@
 	)
 	(segment
-		(start 145.75 73.8138)
-		(end 144.2945 75.2693)
-		(width 0.25)
-		(layer "F.Cu")
-		(net 32)
-	)
-	(segment
 		(start 107.8 117.6)
 		(end 108.8 116.6)
@@
 	)
 	(segment
+		(start 145.75 73.8138)
+		(end 145.75 71.15)
+		(width 0.25)
+		(layer "F.Cu")
+		(net 32)
+	)
+	(segment
 		(start 108.8 116.6)
 		(end 108.8 115.3)
@@
 	)
 	(segment
+		(start 144.771475 74.792325)
+		(end 145.75 73.8138)
+		(width 0.25)
+		(layer "F.Cu")
+		(net 32)
+	)
+	(segment
 		(start 114.35 117.6)
 		(end 114.75 117.2)
@@
 	)
 	(via
-		(at 144.2945 75.2693)
+		(at 144.771475 74.792325)
 		(size 0.6)
 		(drill 0.3)
@@
 	)
 	(segment
-		(start 140.3307 75.2693)
-		(end 144.2945 75.2693)
+		(start 144.2945 75.2693)
+		(end 140.3307 75.2693)
 		(width 0.2)
 		(layer "B.Cu")
@@
 	)
 	(segment
-		(start 129.925 94.4)
+		(start 115.775 116.175)
+		(end 114.75 117.2)
+		(width 0.2)
+		(layer "B.Cu")
+		(net 32)
+	)
+	(segment
+		(start 138.15 93.800001)
 		(end 137.550001 94.4)
 		(width 0.2)
@@
 	)
 	(segment
-		(start 114.75 117.2)
-		(end 115.775 116.175)
+		(start 138.15 77.45)
+		(end 138.15 93.800001)
 		(width 0.2)
 		(layer "B.Cu")
@@
 	(segment
 		(start 137.550001 94.4)
-		(end 138.15 93.800001)
+		(end 129.925 94.4)
 		(width 0.2)
 		(layer "B.Cu")
@@
 	)
 	(segment
-		(start 138.15 77.45)
-		(end 140.3307 75.2693)
+		(start 144.771475 74.792325)
+		(end 144.2945 75.2693)
 		(width 0.2)
 		(layer "B.Cu")
@@
 	(segment
 		(start 115.775 108.55)
-		(end 129.925 94.4)
+		(end 115.775 116.175)
 		(width 0.2)
 		(layer "B.Cu")
@@
 	)
 	(segment
-		(start 138.15 93.800001)
+		(start 140.3307 75.2693)
 		(end 138.15 77.45)
 		(width 0.2)
@@
 	)
 	(segment
-		(start 115.775 116.175)
+		(start 129.925 94.4)
 		(end 115.775 108.55)
 		(width 0.2)
@@
 	)
 	(segment
-		(start 144.9195 75.528184)
-		(end 144.553384 75.8943)
+		(start 145.5 74.636396)
+		(end 145.5 75.5)
 		(width 0.25)
 		(layer "B.Cu")
@@
 	)
 	(segment
-		(start 144.9195 74.8445)
-		(end 144.9195 75.528184)
+		(start 145.5 75.5)
+		(end 145.1057 75.8943)
 		(width 0.25)
 		(layer "B.Cu")
@@
 	)
 	(segment
-		(start 138.65 93.901041)
-		(end 137.726041 94.825)
+		(start 124.825 102.108308)
+		(end 124.825 113.6)
 		(width 0.25)
 		(layer "B.Cu")
@@
 	)
 	(segment
-		(start 142.0876 72.0126)
-		(end 144.9195 74.8445)
+		(start 138.65 93.901041)
+		(end 137.726041 94.825)
 		(width 0.25)
 		(layer "B.Cu")
@@
 	)
 	(segment
-		(start 137.726041 94.825)
-		(end 132.108308 94.825)
+		(start 140.8057 75.8943)
+		(end 138.65 78.05)
 		(width 0.25)
 		(layer "B.Cu")
@@
 	)
 	(segment
-		(start 124.825 102.108308)
-		(end 124.825 113.6)
+		(start 138.65 78.05)
+		(end 138.65 93.901041)
 		(width 0.25)
 		(layer "B.Cu")
@@
 	)
 	(segment
-		(start 144.553384 75.8943)
-		(end 140.8057 75.8943)
+		(start 137.726041 94.825)
+		(end 132.108308 94.825)
 		(width 0.25)
 		(layer "B.Cu")
@@
 	)
 	(segment
-		(start 138.65 78.05)
-		(end 138.65 93.901041)
+		(start 132.108308 94.825)
+		(end 124.825 102.108308)
 		(width 0.25)
 		(layer "B.Cu")
@@
 	)
 	(segment
-		(start 142.0876 62.0972)
-		(end 142.0876 72.0126)
+		(start 145.1057 75.8943)
+		(end 140.8057 75.8943)
 		(width 0.25)
 		(layer "B.Cu")
@@
 	)
 	(segment
-		(start 140.8057 75.8943)
-		(end 138.65 78.05)
+		(start 142.0876 71.223996)
+		(end 145.5 74.636396)
 		(width 0.25)
 		(layer "B.Cu")
@@
 	)
 	(segment
-		(start 132.108308 94.825)
-		(end 124.825 102.108308)
+		(start 142.0876 62.0972)
+		(end 142.0876 71.223996)
 		(width 0.25)
 		(layer "B.Cu")
